File: Hardware/dac.kicad_pcb (KiCad board)
At the start: 2 copper layers, 65 x 100 mm, 114 parts, among them CON1 SD_Card, P1 ANALOG_POWER, P11 JACK, P12 S/PDIF, P13 TORX147, P2 DIGITAL_POWER, P3 ENCODER, P4 SWDIO, P5 UART, P6 OLED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

Commit message: PCB bugfixes.
Routing:
- net GNDD: track 198.2 -> 211.4 mm, vias 7 -> 15
- net +5V: track 124.3 -> 121.9 mm
- net +3V3: track 336.9 -> 339.0 mm
- net Net-(P4-Pad2): track 19.0 -> 21.0 mm, vias 0 -> 2
- net Net-(P4-Pad1): track 23.3 -> 25.0 mm
- net Net-(C19-Pad2): track 15.5 -> 16.1 mm
- net /DAC/~RST: track 150.2 -> 150.7 mm
Other:
- net class Default: clearance 0.2032 -> 0.1524
- rule trace_clearance: 0.2032 -> 0.1524
